File: power_converter/buck.sch (KiCad schematic (older format))
At the start: 46 parts, among them J8 Conn_01x01, J9 Conn_01x01, Q1 Q_PMOS_GDS, U13 LTC2946CMS#PBF

Commit message: Backplane
Deleted full system pwer monitor
Parts:
- removed C20, C21: .1uF, Capacitors_SMD:C_0805, symbol Device:C_Small
- removed R47: WSLP59311L000FEB, rov:WSLP59311L000FEB, symbol rov:WSLP59311L000FEB
- removed R50: 4.7K, Resistors_SMD:R_1206, symbol Device:R_US
- removed U13: LTC2946CMS#PBF, Housings_SSOP:MSOP-16_3x4mm_Pitch0.5mm, symbol rov:LTC2946CMS#PBF
Connections:
- net labels added: 12P
- net labels removed: GP_OUTPUT, SCL_iso, SDA_iso
- wire segments 165 -> 134
- no-connect marks 3 -> 2
Other:
- note removed: "102.4mV max sense voltage differential\n@100A, this equates to 1.024mOhm@10W power rating\n"
- note removed: "Power Monitor"
