File: backplane.kicad_pcb (KiCad board)
At the start: 4 copper layers, 113.5 x 84 mm, 140 parts, among them J1 Conn_01x01, J1 Conn_01x02, J2 Conn_01x02, J2 Conn_01x03_Female, J2 PCA, J3 Bar02, J4 Conn_01x02, J4 LSM303, J5 Conn_01x02, J6 LSM303, Q1 Q_PMOS_GDS, U1 LTC2946CMS#PBF, U1 SCA3300, U10 TSC888, U11 TSC888, U12 TSC888, U2 MAX6581, U3 LM3480-3.3, U3 MAX6581, U4 ADuM1250, U4 LTC2946CMS#PBF, U5 ADuM1250, U5 LM3480-3.3, U6 PI_ZERO, U7 TSC888, U8 TSC888, U9 TSC888

Commit message: PCA symbol moved to sensor board
Parts:
- added 1.6k1: R_Small, Resistor_SMD:R_0805_2012Metric_Pad1.15x1.40mm_HandSolder, F.Cu at (191.2, 40.4)
- added 1.6k2: R_Small, Resistor_SMD:R_0805_2012Metric_Pad1.15x1.40mm_HandSolder, F.Cu at (191.2, 44.8)
- added C24: 0.01u, Capacitor_SMD:C_0805_2012Metric_Pad1.15x1.40mm_HandSolder, F.Cu at (196.8, 51.2)
- added C25: 0.1u, Capacitor_SMD:C_0805_2012Metric_Pad1.15x1.40mm_HandSolder, F.Cu at (193.7, 51.2)
- added C26: 0.01u, Capacitor_SMD:C_0805_2012Metric_Pad1.15x1.40mm_HandSolder, F.Cu at (201.2, 51.2)
- added C27: 0.1u, Capacitor_SMD:C_0805_2012Metric_Pad1.15x1.40mm_HandSolder, F.Cu at (204.2, 51.2)
- added R13: 1.6k, Resistor_SMD:R_0805_2012Metric_Pad1.15x1.40mm_HandSolder, F.Cu at (206.4, 40.4)
- added R14: 1.6k, Resistor_SMD:R_0805_2012Metric_Pad1.15x1.40mm_HandSolder, F.Cu at (206.4, 45.0)
- added U5: ADuM1250, Package_SO:SO-8_5.3x6.2mm_P1.27mm, F.Cu at (199.0, 42.6)
- added U6: PI_ZERO, rov:PI_ZERO, F.Cu at (240.6, 43.8)
- moved C3 199.1 mm to (228.7, 126.0)
- moved C4 199.1 mm to (221.6, 136.6)
- moved C6 199.1 mm to (237.4, 127.2)
- moved C7 199.1 mm to (237.4, 129.6)
- moved J2 199.1 mm to (230.9, 146.9)
- moved J3 199.1 mm to (237.2, 141.5)
- moved U3 199.1 mm to (229.9, 131.1)
- moved U5 199.1 mm to (237.3, 123.9)
- moved C5 199.1 mm to (231.2, 136.6)
- moved J1 199.1 mm to (221.2, 146.9)
- moved J4 199.1 mm to (212.1, 141.2)
- moved U4 199.1 mm to (218.7, 130.8)
- moved BC4 34.6 mm to (154.9, 32.7)
- moved R7 34.6 mm to (166.9, 66.9)
- moved BC1 34.6 mm to (82.5, 54.9)
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Routing:
- net Net-(R14-Pad2): track 0.00 -> 39.6 mm
- net Net-(R13-Pad2): track 0.00 -> 39.3 mm
- net /VOUT: vias 69 -> 66
- net +5VP: vias 17 -> 18
- net 5VPI: vias 1 -> 2
- net /SCL_iso: vias 0 -> 1
Other:
- net class Default: trace_width 0.5 -> 0.25

Commit message: updated library
Parts:
- removed the C10 at (152.5, 40.4)
- removed the C11 at (150.0, 40.4)
- removed the C12 at (165.0, 20.9)
- removed the C3 at (150.5, 58.2)
- removed the C4 at (142.0, 58.9)
- removed the C4 at (221.6, 136.6)
- removed the C5 at (138.0, 58.9)
- removed the C5 at (231.2, 136.6)
- removed the C6 at (154.0, 34.9)
- removed the C6 at (237.4, 127.2)
- removed the C7 at (154.0, 32.4)
- removed the C7 at (237.4, 129.6)
- removed the C8 at (152.5, 69.9)
- removed the C9 at (155.0, 69.9)
- removed D8: LED, LEDs:LED_0805
- removed the J1 at (75.0, 23.4)
- removed the J1 at (221.2, 146.9)
- removed the J2 at (75.0, 91.4)
- removed the J2 at (230.9, 146.9)
- removed the J3 at (114.8, 185.6)
- removed the J3 at (237.2, 141.5)
- removed JP1, JP2, JP3, JP4: SolderJumper_2_Open, jumpers:SolderJumper-2_P1.3mm_Open_RoundedPad1.0x1.5mm
- removed the R1 at (72.0, 56.4)
- removed the R10 at (94.7, 22.2)
- removed the R11 at (181.6, 70.2)
- removed the R12 at (145.0, 35.9)
- removed the R13 at (155.6, 96.9)
- removed the R2 at (76.6, 81.4)
- removed the R3 at (167.5, 85.8)
- removed the R4 at (134.0, 58.9)
- removed the R5 at (165.4, 51.9)
- removed the R6 at (167.1, 71.9)
- removed the R7 at (166.9, 66.9)
- removed the R8 at (156.5, 66.4)
- removed the R9 at (185.7, 12.4)
- removed TP1, TP2: TestPoint, Measurement_Points:Measurement_Point_Square-TH_Small
- removed the U3 at (229.9, 131.1)
- removed the U4 at (218.7, 130.8)
- removed the U5 at (237.3, 123.9)
- added C13: 10uF, rov:C_2220_SMD, F.Cu at (-203.5, 146.6)
- added C14: 100uF, rov:PCR1J101MCL1GS, F.Cu at (-204.0, 162.6)
- added C15: 330uF, rov:PCR1J101MCL1GS, F.Cu at (-122.7, 141.6)
- added C16: 10uF, rov:C_1206_SMD, F.Cu at (-123.7, 123.6)
- added C17: 1uF, rov:C_1206_SMD, F.Cu at (-123.7, 132.6)
- added C18: 2.2uF, rov:C_0805_SMD, F.Cu at (-121.8, 160.6)
- added C19: 2.2uF, rov:C_0805_SMD, F.Cu at (-118.2, 160.6)
- added C22: 10uF, rov:C_1206_SMD, F.Cu at (-109.2, 157.6)
- added C23: 1uF, rov:C_1206_SMD, F.Cu at (-109.2, 161.0)
- added C28: 47uF, rov:C_1206_SMD, F.Cu at (-109.2, 150.4)
- added C4: 0.1uF, Capacitor_SMD:C_0805_2012Metric_Pad1.15x1.40mm_HandSolder, F.Cu at (-58.9, 174.1)
- added C5: 0.1uF, Capacitor_SMD:C_0805_2012Metric_Pad1.15x1.40mm_HandSolder, F.Cu at (-56.7, 174.3)
- added J1: Bar02, Connector_PinHeader_2.54mm:PinHeader_1x04_P2.54mm_Vertical, F.Cu at (-42.4, 177.6)
- added J2: Conn_02x15_Top_Bottom, rov:PCA9685, F.Cu at (-80.9, 130.0)
- added J3: Conn_01x03_Female, ROV:Wago Terminal Blocks, F.Cu at (-226.8, 85.8)
- added J3: Conn_01x02, Connector_JST:JST_EH_B02B-EH-A_1x02_P2.50mm_Vertical, F.Cu at (-58.5, 184.8)
- added J5: LSM303, rov:LSM303, F.Cu at (-89.8, 186.5)
- added J8: Conn_01x01, rov:7466004, F.Cu at (-220.0, 123.1)
- added J9: Conn_01x01, rov:7466004, F.Cu at (-220.0, 147.1)
- added R43: 100k, rov:R_1206_SMD, F.Cu at (-209.0, 140.6)
- added R44: 12K, rov:R_1206_SMD, F.Cu at (-204.0, 153.1)
- added R45: 470K, rov:R_1206_SMD, F.Cu at (-126.6, 106.0)
- added R46: 3.3K, rov:C_1206_SMD, F.Cu at (-123.7, 128.1)
- added R51: 2.4K, rov:C_1206_SMD, F.Cu at (-216.5, 109.3)
- added R52: 600, rov:C_1206_SMD, F.Cu at (39.6, 267.0)
- added R53: 600, rov:C_1206_SMD, F.Cu at (39.4, 258.5)
- added R54: 600, rov:C_1206_SMD, F.Cu at (39.4, 261.9)
- added U2: LM3480-3.3, Package_TO_SOT_SMD:SOT-23, F.Cu at (-62.2, 174.1)
- BC1, BC2, BC4: moved to F.Cu
- C1: value 100nF -> .1uF
- C1: value 10uF -> 100pF; footprint Capacitors_SMD:C_2220 -> Capacitor_SMD:C_0805_2012Metric_Pad1.15x1.40mm_HandSolder
- C2: value 100nF -> 100pF; footprint rov:PCR1J101MCL1GS -> Capacitor_SMD:C_0805_2012Metric_Pad1.15x1.40mm_HandSolder
- C9: value 0.1uF -> 10nF
- D1: footprint Diodes_SMD:D_SOD-123 -> Diode_SMD:D_SOD-123
- D2: footprint Diodes_SMD:D_SOD-123F -> rov:D_SOD-123F
- D3: footprint Diodes_SMD:D_SMB -> rov:D_SOD-123F
- D4, D5, D6, D7: footprint LEDs:LED_0805 -> LED_SMD:LED_0805_2012Metric_Pad1.15x1.40mm_HandSolder
- F1: footprint Resistors_SMD:R_1812 -> rov:R_1812_SMD
- J1, J4, J5: value Conn_01x02 -> Conn_01x03_Female
- J4: value LSM303 -> Conn_01x02; footprint Connector_PinHeader_2.54mm:PinHeader_1x08_P2.54mm_Vertical -> Connector_JST:JST_EH_B02B-EH-A_1x02_P2.50mm_Vertical
- J6: value LSM303 -> Conn_01x03_Female
- Q1: footprint TO_SOT_Packages_SMD:TO-263-2 -> Package_TO_SOT_SMD:TO-263-2
- R1: value 100k -> WSLP59311L000FEB
- R14: value 1.6k -> 100
- R9: value 2.4K -> 10k
- U1: value SCA3300 -> PIC16F15323
- U1: value LTC2946CMS#PBF -> MAX6581; footprint Housings_SSOP:MSOP-16_3x4mm_Pitch0.5mm -> Package_DFN_QFN:QFN-20-1EP_5x5mm_P0.65mm_EP3.35x3.35mm
- U2: value MAX6581 -> PIC16F15323
- U3: value LM3480-3.3 -> PIC16F15323
- U4: value LTC2946CMS#PBF -> PIC16F15323
- U5: value ADuM1250 -> PIC16F15323
- U6: value PI_ZERO -> PIC16F15323
- moved J1 426.2 mm to (-227.2, 31.2), turned to 90 degrees
- moved D4 418.2 mm to (-222.1, 109.3), turned to 180 degrees
- moved J2 389.3 mm to (-227.2, 58.9), turned to 90 degrees
- moved ESC1 375.4 mm to (-193.5, 17.6), turned to 180 degrees
- moved U7 361.4 mm to (-174.6, 33.3), turned to 270 degrees
- moved R1 352.5 mm to (-176.4, 16.3), turned to 180 degrees
- moved R9 346.3 mm to (-164.8, 27.4), turned to 0 degrees
- moved R15 340.2 mm to (-159.9, 27.4), turned to 180 degrees
- moved C9 338.2 mm to (-159.8, 24.6), turned to 0 degrees
- moved ESC2 337.5 mm to (-192.1, 44.4), turned to 180 degrees
- moved U1 327.1 mm to (-153.9, 18.9), turned to 0 degrees
- moved U8 324.3 mm to (-173.3, 58.3), turned to 270 degrees
- moved R22 323.9 mm to (-142.2, 34.5), turned to 180 degrees
- moved C1 322.4 mm to (-152.8, 13.9), turned to 0 degrees
- moved R21 322.0 mm to (-142.2, 31.9), turned to 180 degrees
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Connections:
- BC1 pad 1: /Power Conversion/VIN+ -> /VIN+
- BC1 pad 9: /Power Conversion/VOUT -> +12P
- BC2 pad 1: /Power Conversion/VIN+ -> /VIN+
- BC2 pad 9: /Power Conversion/VOUT -> +12P
- C1 pad 1: Net-(C1-Pad1) -> +5VP
- C1 pad 2: +3V3 -> GNDPWR
- C1 pad 1: /VIN+ -> /temp1p
- C1 pad 2: Earth -> /temp1n
- C2 pad 1: Net-(C2-Pad1) -> /temp2p
- C2 pad 2: +3V3 -> /temp2n
- C9 pad 1: +3V3 -> Net-(C9-Pad1)
- C9 pad 2: GNDS -> GNDPWR
- D1 pad 1: /Power Conversion/VIN+ -> /VIN+
- D5 pad 2: /Power Conversion/VOUT -> +12P
- J1 pad 1: /SCL -> Net-(ESC1-Pad5)
- J1 pad 2: /SDA -> Net-(ESC1-Pad6)
- J1 pad 3: (no net) -> Net-(ESC1-Pad7)
- J4 pad 1: /Sensor Breakout/temp1p -> Net-(ESC4-Pad5)
- J4 pad 2: /Sensor Breakout/temp1n -> Net-(ESC4-Pad6)
- J4 pad 3: (no net) -> Net-(ESC4-Pad7)
- J4 pad 1: /SCL1 -> /temp2p
- J4 pad 2: /SDA1 -> /temp2n
- J5 pad 1: /Sensor Breakout/temp2p -> Net-(ESC5-Pad5)
- J5 pad 2: /Sensor Breakout/temp2n -> Net-(ESC5-Pad6)
- J5 pad 3: (no net) -> Net-(ESC5-Pad7)
- J6 pad 1: /Sensor Breakout/SCL1 -> Net-(ESC6-Pad5)
- J6 pad 2: /Sensor Breakout/SDA1 -> Net-(ESC6-Pad6)
- J6 pad 3: /Sensor Breakout/I2 -> Net-(ESC6-Pad7)
- Q1 pad 3: /Power Conversion/VIN+ -> /VIN+
- R1 pad 1: Net-(D1-Pad2) -> +12P
- R1 pad 2: Earth -> Net-(ESC1-Pad1)
- R14 pad 1: 5VPI -> Net-(R14-Pad1)
- R14 pad 2: Net-(R14-Pad2) -> Net-(C8-Pad1)
- R9 pad 1: Earth -> +5VP
- R9 pad 2: Net-(D4-Pad1) -> Net-(C9-Pad1)
- U1 pad 1: GNDS -> +5VP
- U1 pad 10: Net-(C4-Pad2) -> Net-(R20-Pad2)
- U1 pad 11: GNDS -> Net-(R19-Pad2)
- U1 pad 12: GNDS -> Net-(U1-Pad12)
- U1 pad 13: (no net) -> Net-(U1-Pad13)
- U1 pad 14: (no net) -> GNDPWR
- U1 pad 2: Net-(C1-Pad1) -> GNDPWR
- U1 pad 3: Net-(U1-Pad3) -> GNDPWR
- U1 pad 4: Net-(C2-Pad1) -> Net-(R15-Pad1)
- U1 pad 5: +3V3 -> GNDPWR
- U1 pad 6: /Sensor Breakout/MISO -> /CS1
- U1 pad 7: /Sensor Breakout/MOSI -> /PWM1
- U1 pad 8: /Sensor Breakout/SCK -> Net-(R22-Pad2)
- U1 pad 9: Net-(C5-Pad2) -> Net-(R21-Pad2)
- U1 pad 1: /VOUT -> /temp1n
- U1 pad 10: Net-(U1-Pad10) -> (no net)
- U1 pad 11: GNDPWR -> (no net)
- U1 pad 12: /ADR0 -> (no net)
- U1 pad 13: /VOUT -> (no net)
- U1 pad 14: /ADR1 -> (no net)
- U1 pad 15: +12P -> (no net)
- U1 pad 16: /VOUT -> (no net)
- U1 pad 2: /INTVCC -> /temp1p
- U1 pad 3: /GP_OUTPUT -> /temp2n
- U1 pad 4: GNDPWR -> /temp2p
- U1 pad 5: GNDPWR -> (no net)
- U1 pad 6: /SDAISO -> (no net)
- U1 pad 7: /SDAISO -> (no net)
- U1 pad 8: /SCLISO -> (no net)
- U1 pad 9: GNDPWR -> (no net)
- U2 pad 1: /Sensor Breakout/temp1n -> +5VP
- U2 pad 10: (no net) -> Net-(R24-Pad2)
- U2 pad 11: (no net) -> Net-(R23-Pad2)
- U2 pad 12: (no net) -> Net-(U2-Pad12)
- U2 pad 13: (no net) -> Net-(U2-Pad13)
- U2 pad 14: (no net) -> GNDPWR
- U2 pad 2: /Sensor Breakout/temp1p -> +5VP
- U2 pad 3: /Sensor Breakout/temp2n -> GNDPWR
- U2 pad 4: /Sensor Breakout/temp2p -> Net-(R13-Pad1)
- U2 pad 5: (no net) -> GNDPWR
- U2 pad 6: (no net) -> /CS2
- U2 pad 7: (no net) -> /PWM2
- U2 pad 8: (no net) -> Net-(R26-Pad2)
- U2 pad 9: (no net) -> Net-(R25-Pad2)
- U3 pad 1: +3V3 -> +5VP
- U3 pad 10: (no net) -> Net-(R28-Pad2)
- U3 pad 11: (no net) -> Net-(R27-Pad2)
- U3 pad 12: (no net) -> Net-(U3-Pad12)
- U3 pad 13: (no net) -> Net-(U3-Pad13)
- U3 pad 14: (no net) -> GNDPWR
- U3 pad 2: +12P -> GNDPWR
- U3 pad 3: GND -> +5VP
- U3 pad 4: (no net) -> Net-(R14-Pad1)
- U3 pad 5: (no net) -> GNDPWR
- U3 pad 6: (no net) -> /CS3
- U3 pad 7: (no net) -> /PWM3
- U3 pad 8: (no net) -> Net-(R30-Pad2)
- U3 pad 9: (no net) -> Net-(R29-Pad2)
- U4 pad 1: /Power Conversion/VOUT -> +5VP
- U4 pad 10: Net-(U4-Pad10) -> Net-(R32-Pad2)
- U4 pad 11: GNDPWR -> Net-(R31-Pad2)
- U4 pad 12: /Power Conversion/ADR0 -> Net-(U4-Pad12)
- U4 pad 13: /Power Conversion/VOUT -> Net-(U4-Pad13)
- U4 pad 14: /Power Conversion/ADR1 -> GNDPWR
- U4 pad 2: /Power Conversion/INTVCC -> +5VP
- U4 pad 3: /Power Conversion/GP_OUTPUT -> +5VP
- U4 pad 4: GNDPWR -> Net-(R16-Pad1)
- U4 pad 6: /Power Conversion/SDA_iso -> /CS4
- U4 pad 7: /Power Conversion/SDA_iso -> /PWM4
- U4 pad 8: /Power Conversion/SCL_iso -> Net-(R34-Pad2)
- U4 pad 9: GNDPWR -> Net-(R33-Pad2)
- U5 pad 10: (no net) -> Net-(R36-Pad2)
- U5 pad 11: (no net) -> Net-(R35-Pad2)
- U5 pad 12: (no net) -> Net-(U5-Pad12)
- U5 pad 13: (no net) -> Net-(U5-Pad13)
- U5 pad 14: (no net) -> GNDPWR
- U5 pad 2: /Pi/SDA_iso -> GNDPWR
- U5 pad 3: /Pi/SCL_iso -> GNDPWR
- U5 pad 4: GNDPWR -> Net-(R17-Pad1)
- U5 pad 5: GNDS -> +5VP
- U5 pad 6: Net-(R14-Pad2) -> /CS5
- U5 pad 7: Net-(R13-Pad2) -> /PWM5
- U5 pad 8: 5VPI -> Net-(R38-Pad2)
- U5 pad 9: (no net) -> Net-(R37-Pad2)
- U6 pad 1: +3V3 -> +5VP
- U6 pad 10: Net-(U6-Pad10) -> Net-(R40-Pad2)
- U6 pad 11: Net-(U6-Pad11) -> Net-(R39-Pad2)
- U6 pad 14: GNDS -> GNDPWR
- U6 pad 2: 5VPI -> +5VP
- U6 pad 3: Net-(R13-Pad2) -> GNDPWR
- U6 pad 4: 5VPI -> Net-(R18-Pad1)
- U6 pad 5: Net-(R14-Pad2) -> +5VP
- U6 pad 6: GNDS -> /CS6
- U6 pad 7: Net-(U6-Pad7) -> /PWM6
- U6 pad 8: Net-(U6-Pad8) -> Net-(R42-Pad2)
- U6 pad 9: GNDS -> Net-(R41-Pad2)
Routing:
- net +5VP: track 50.8 -> 159.5 mm, vias 18 -> 51
- net /SCL1: track 60.0 -> 0.00 mm, vias 2 -> 0
- net /SDA1: track 50.9 -> 0.00 mm, vias 2 -> 0
- net +3V3: track 30.3 -> 78.4 mm, vias 4 -> 0
- net +12P: track 107.7 -> 70.2 mm, vias 31 -> 64
- net Net-(R14-Pad2): track 39.6 -> 7.24 mm
- net Net-(R13-Pad2): track 39.3 -> 7.24 mm
- net /INTVCC: track 31.6 -> 0.00 mm, vias 2 -> 0
- net /VOUT: track 25.7 -> 0.00 mm, vias 66 -> 0
- net Net-(ESC1-Pad1): track 18.2 -> 0.00 mm
- net GNDS: track 9.31 -> 26.6 mm, vias 6 -> 2
- net Net-(BC4-Pad22): track 0.00 -> 16.6 mm
- net +5V: track 3.42 -> 18.5 mm
- net /GP_OUTPUT: track 11.2 -> 0.00 mm
- net Earth: track 12.5 -> 2.34 mm, vias 40 -> 13
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- removed copper zone on power.Cu, net +3V3
- removed copper zone on F.Cu, net +5V
- removed copper zone on F.Cu, net /VOUT
- removed copper zone on power.Cu, net /VOUT
- removed copper zone on F.Cu, net 5VPI
- removed copper zone on ground.Cu, net GND
- removed copper zone on B.Cu, net GNDPWR
- removed copper zone on F.Cu, net GNDS
Other:
- board outline removed
- board text removed: "0"
- board text removed: "1"
- board text removed: "12V PWR GOOD"
- board text removed: "48V PWR GOOD"
- board text removed: "5V ISO GOOD"
- board text removed: "DESIGNED FOR 2 OZ COPPER EXTERNAL/1.5OZ COPPER INTERNAL ASSUMING ~1 mil HASL W/LEAD SURFACE FINISH"
- board text removed: "NUGGET Industries PDB REV 1A"
- board text removed: "SET i2c ADDRESS WITH SOLDER PADS."
- board text removed: "rPI INPUT PROTECTION"
- board text removed: "top trace 2oz sized for 50a using matlab calculator, confirmed ballpark with saturn in1 derated 30% for internal layer sizing, matlab and saturn minimum vias for 100a at 25 drill and 50 ring size is 46, there are 50+ vias"
