File: power_v2/buck.sch (KiCad schematic (older format))
At the start: 41 parts, among them J8 Conn_01x01, J9 Conn_01x01, Q1 Q_PMOS_GDS

Commit message: PCA symbol moved to sensor board
Parts:
- removed JP1, JP2, JP3, JP4: SolderJumper_2_Open, jumpers:SolderJumper-2_P1.3mm_Open_RoundedPad1.0x1.5mm, symbol Jumper:SolderJumper_2_Open
- removed R48, R49: 22K, Resistors_SMD:R_1206, symbol Device:R_US
Connections:
- net labels removed: ADR0, ADR1, INTVCC
- wire segments 134 -> 120
Other:
- note removed: "i2c Address Bits\nTri-State Address\n(see datasheet)\n"
