File: power_alec/buck.sch (KiCad schematic (older format))
At the start: 35 parts, among them J8 Conn_01x01, J9 Conn_01x01, Q1 Q_PMOS_GDS

Commit message: not much
Parts:
- C13: footprint Capacitors_SMD:C_2220 -> rov:C_2220_SMD
- C16, C17, C22, C23, C28: footprint Capacitors_SMD:C_1206 -> rov:C_1206_SMD
- C18, C19: footprint Capacitors_SMD:C_0805 -> rov:C_0805_SMD
- D1: footprint Diodes_SMD:D_SOD-123 -> Diode_SMD:D_SOD-123
- D2: footprint Diodes_SMD:D_SOD-123F -> rov:D_SOD-123F
- D3: footprint Diodes_SMD:D_SMB -> rov:D_SOD-123F
- D4, D5, D6, D7: footprint LEDs:LED_0805 -> LED_SMD:LED_0805_2012Metric_Pad1.15x1.40mm_HandSolder
- F1: footprint Resistors_SMD:R_1812 -> rov:R_1812_SMD
- Q1: footprint TO_SOT_Packages_SMD:TO-263-2 -> Package_TO_SOT_SMD:TO-263-2
- R43, R44, R45: footprint Resistors_SMD:R_1206 -> rov:R_1206_SMD
- R46, R51, R52, R53, R54: footprint Resistors_SMD:R_1206 -> rov:C_1206_SMD
Connections:
- net labels removed: 12P
Changed lines of the file:
@@
 F 0 "R44" H 3568 3246 50  0000 L CNN
 F 1 "12K" H 3568 3155 50  0000 L CNN
-F 2 "Resistors_SMD:R_1206" V 3540 3190 50  0001 C CNN
+F 2 "rov:R_1206_SMD" V 3540 3190 50  0001 C CNN
 F 3 "~" H 3500 3200 50  0001 C CNN
 	1    3500 3200
@@
 F 0 "C13" H 2842 3246 50  0000 L CNN
 F 1 "10uF" H 2842 3155 50  0000 L CNN
-F 2 "Capacitors_SMD:C_2220" H 2750 3200 50  0001 C CNN
+F 2 "rov:C_2220_SMD" H 2750 3200 50  0001 C CNN
 F 3 "http://datasheets.avx.com/X7RDielectric.pdf" H 2750 3200 50  0001 C CNN
 F 4 "22201C106MAT2A" H 2750 3200 50  0001 C CNN "PN"
@@
 F 0 "C16" V 5971 2600 50  0000 C CNN
 F 1 "10uF" V 6062 2600 50  0000 C CNN
-F 2 "Capacitors_SMD:C_1206" H 6200 2600 50  0001 C CNN
+F 2 "rov:C_1206_SMD" H 6200 2600 50  0001 C CNN
 F 3 "http://www.samsungsem.com/kr/support/product-search/mlcc/__icsFiles/afieldfile/2018/07/19/CL31B106KLHNFNE.pdf" H 6200 2600 50  0001 C CNN
 F 4 "CL31B106KLHNFNE" V 6200 2600 50  0001 C CNN "PN"
@@
 F 0 "C17" V 6321 2600 50  0000 C CNN
 F 1 "1uF" V 6412 2600 50  0000 C CNN
-F 2 "Capacitors_SMD:C_1206" H 6550 2600 50  0001 C CNN
+F 2 "rov:C_1206_SMD" H 6550 2600 50  0001 C CNN
 F 3 "" H 6550 2600 50  0001 C CNN
 	1    6550 2600
@@
 F 0 "Q1" V 2393 2550 50  0000 C CNN
 F 1 "Q_PMOS_GDS" V 2302 2550 50  0000 C CNN
-F 2 "TO_SOT_Packages_SMD:TO-263-2" H 2250 2650 50  0001 C CNN
+F 2 "Package_TO_SOT_SMD:TO-263-2" H 2250 2650 50  0001 C CNN
 F 3 "https://www.infineon.com/dgdl/SPB80P06P+G_Rev+1.6_.pdf?folderId=db3a304412b407950112b408e8c90004&fileId=db3a304412b407950112b42add964408" H 2050 2550 50  0001 C CNN
 F 4 "SPB80P06PGATMA1" V 2050 2550 50  0001 C CNN "PN"
@@
 F 0 "D1" V 2304 2679 50  0000 L CNN
 F 1 "12V" V 2395 2679 50  0000 L CNN
-F 2 "Diodes_SMD:D_SOD-123" H 2350 2600 50  0001 C CNN
+F 2 "Diode_SMD:D_SOD-123" H 2350 2600 50  0001 C CNN
 F 3 "http://www.mccsemi.com/up_pdf/MMSZ5221-MMSZ5261(SOD123).pdf" H 2350 2600 50  0001 C CNN
 F 4 "MMSZ5245B-TP" V 2350 2600 50  0001 C CNN "PN"
@@
 F 0 "R43" H 2118 3246 50  0000 L CNN
 F 1 "100k" H 2118 3155 50  0000 L CNN
-F 2 "Resistors_SMD:R_1206" V 2090 3190 50  0001 C CNN
+F 2 "rov:R_1206_SMD" V 2090 3190 50  0001 C CNN
 F 3 "~" H 2050 3200 50  0001 C CNN
 	1    2050 3200
@@
 F 0 "D5" H 10242 1445 50  0000 C CNN
 F 1 "LED" H 10242 1536 50  0000 C CNN
-F 2 "LEDs:LED_0805" H 10250 1700 50  0001 C CNN
+F 2 "LED_SMD:LED_0805_2012Metric_Pad1.15x1.40mm_HandSolder" H 10250 1700 50  0001 C CNN
 F 3 "~" H 10250 1700 50  0001 C CNN
 F 4 "LG R971-KN-1" H 10250 1700 50  0001 C CNN "PN"
@@
 F 0 "R52" V 10395 1700 50  0000 C CNN
 F 1 "600" V 10486 1700 50  0000 C CNN
-F 2 "Resistors_SMD:R_1206" V 10640 1690 50  0001 C CNN
+F 2 "rov:C_1206_SMD" V 10640 1690 50  0001 C CNN
 F 3 "~" H 10600 1700 50  0001 C CNN
 	1    10600 1700
@@
 F 0 "R46" H 6868 2646 50  0000 L CNN
 F 1 "3.3K" H 6868 2555 50  0000 L CNN
-F 2 "Resistors_SMD:R_1206" V 6840 2590 50  0001 C CNN
+F 2 "rov:C_1206_SMD" V 6840 2590 50  0001 C CNN
 F 3 "~" H 6800 2600 50  0001 C CNN
 	1    6800 2600
@@
 F 0 "C22" V 8521 5800 50  0000 C CNN
 F 1 "10uF" V 8612 5800 50  0000 C CNN
-F 2 "Capacitors_SMD:C_1206" H 8750 5800 50  0001 C CNN
+F 2 "rov:C_1206_SMD" H 8750 5800 50  0001 C CNN
 F 3 "http://www.samsungsem.com/kr/support/product-search/mlcc/__icsFiles/afieldfile/2018/07/19/CL31B106KLHNFNE.pdf" H 8750 5800 50  0001 C CNN
 F 4 "CL31B106KLHNFNE" V 8750 5800 50  0001 C CNN "PN"
@@
 F 0 "C23" V 8871 5800 50  0000 C CNN
 F 1 "1uF" V 8962 5800 50  0000 C CNN
-F 2 "Capacitors_SMD:C_1206" H 9100 5800 50  0001 C CNN
+F 2 "rov:C_1206_SMD" H 9100 5800 50  0001 C CNN
 F 3 "" H 9100 5800 50  0001 C CNN
 	1    9100 5800
@@
 F 0 "C19" V 7300 5700 50  0000 C CNN
 F 1 "2.2uF" V 7100 5700 50  0000 C CNN
-F 2 "Capacitors_SMD:C_0805" H 7200 5700 50  0001 C CNN
+F 2 "rov:C_0805_SMD" H 7200 5700 50  0001 C CNN
 F 3 "?" H 7200 5700 50  0001 C CNN
 F 4 "C2012X7R1C225K125AB" V 7200 5700 50  0001 C CNN "PN"
@@
 F 0 "C18" V 6900 5700 50  0000 C CNN
 F 1 "2.2uF" V 6700 5700 50  0000 C CNN
-F 2 "Capacitors_SMD:C_0805" H 6800 5700 50  0001 C CNN
+F 2 "rov:C_0805_SMD" H 6800 5700 50  0001 C CNN
 F 3 "?" H 6800 5700 50  0001 C CNN
 F 4 "C2012X7R1C225K125AB" V 6800 5700 50  0001 C CNN "PN"
@@
 F 0 "F1" V 10005 5600 50  0000 C CNN
 F 1 "MF-MSMF250/16X-2" V 9914 5600 50  0000 C CNN
-F 2 "Resistors_SMD:R_1812" H 9850 5400 50  0001 L CNN
+F 2 "rov:R_1812_SMD" H 9850 5400 50  0001 L CNN
 F 3 "https://www.bourns.com/docs/Product-Datasheets/mfmsmf.pdf" H 9800 5600 50  0001 C CNN
 	1    9800 5600
@@
 F 0 "D3" V 9954 5868 50  0000 L CNN
 F 1 "SMBJ5.0A-13-F" V 10045 5868 50  0000 L CNN
-F 2 "Diodes_SMD:D_SMB" V 10000 5800 50  0001 C CNN
+F 2 "rov:D_SOD-123F" V 10000 5800 50  0001 C CNN
 F 3 "https://www.diodes.com/assets/Datasheets/ds19002.pdf" V 10000 5800 50  0001 C CNN
 	1    10000 5800
@@
 F 0 "C28" V 10721 5800 50  0000 C CNN
 F 1 "47uF" V 10812 5800 50  0000 C CNN
-F 2 "Capacitors_SMD:C_1206" H 10950 5800 50  0001 C CNN
+F 2 "rov:C_1206_SMD" H 10950 5800 50  0001 C CNN
 F 3 "" H 10950 5800 50  0001 C CNN
 	1    10950 5800
@@
 F 0 "D6" H 10242 1895 50  0000 C CNN
 F 1 "LED" H 10242 1986 50  0000 C CNN
-F 2 "LEDs:LED_0805" H 10250 2150 50  0001 C CNN
+F 2 "LED_SMD:LED_0805_2012Metric_Pad1.15x1.40mm_HandSolder" H 10250 2150 50  0001 C CNN
 F 3 "~" H 10250 2150 50  0001 C CNN
 F 4 "LG R971-KN-1" H 10250 2150 50  0001 C CNN "PN"
@@
 F 0 "R53" V 10395 2150 50  0000 C CNN
 F 1 "600" V 10486 2150 50  0000 C CNN
-F 2 "Resistors_SMD:R_1206" V 10640 2140 50  0001 C CNN
+F 2 "rov:C_1206_SMD" V 10640 2140 50  0001 C CNN
 F 3 "~" H 10600 2150 50  0001 C CNN
 	1    10600 2150
@@
 F 0 "D4" H 10242 995 50  0000 C CNN
 F 1 "LED" H 10242 1086 50  0000 C CNN
-F 2 "LEDs:LED_0805" H 10250 1250 50  0001 C CNN
+F 2 "LED_SMD:LED_0805_2012Metric_Pad1.15x1.40mm_HandSolder" H 10250 1250 50  0001 C CNN
 F 3 "~" H 10250 1250 50  0001 C CNN
 F 4 "LG R971-KN-1" H 10250 1250 50  0001 C CNN "PN"
@@
 F 0 "R51" V 10395 1250 50  0000 C CNN
 F 1 "2.4K" V 10486 1250 50  0000 C CNN
-F 2 "Resistors_SMD:R_1206" V 10640 1240 50  0001 C CNN
+F 2 "rov:C_1206_SMD" V 10640 1240 50  0001 C CNN
 F 3 "~" H 10600 1250 50  0001 C CNN
 	1    10600 1250
@@
 F 0 "D2" H 7900 3687 50  0000 C CNN
 F 1 "D_Small_ALT" H 7900 3686 50  0001 C CNN
-F 2 "Diodes_SMD:D_SOD-123F" V 7900 3800 50  0001 C CNN
+F 2 "rov:D_SOD-123F" V 7900 3800 50  0001 C CNN
 F 3 "http://www.mccsemi.com/up_pdf/SSL16PL(SOD-123FL)-D.pdf" V 7900 3800 50  0001 C CNN
 	1    7900 3800
@@
 F 0 "R45" H 7868 4296 50  0000 L CNN
 F 1 "470K" H 7868 4205 50  0000 L CNN
-F 2 "Resistors_SMD:R_1206" V 7840 4240 50  0001 C CNN
+F 2 "rov:R_1206_SMD" V 7840 4240 50  0001 C CNN
 F 3 "~" H 7800 4250 50  0001 C CNN
 	1    7800 4250
@@
 F 0 "D7" H 10242 2395 50  0000 C CNN
 F 1 "LED" H 10242 2486 50  0000 C CNN
-F 2 "LEDs:LED_0805" H 10250 2650 50  0001 C CNN
+F 2 "LED_SMD:LED_0805_2012Metric_Pad1.15x1.40mm_HandSolder" H 10250 2650 50  0001 C CNN
 F 3 "~" H 10250 2650 50  0001 C CNN
 F 4 "LG R971-KN-1" H 10250 2650 50  0001 C CNN "PN"
@@
 F 0 "R54" V 10395 2650 50  0000 C CNN
 F 1 "600" V 10486 2650 50  0000 C CNN
-F 2 "Resistors_SMD:R_1206" V 10640 2640 50  0001 C CNN
+F 2 "rov:C_1206_SMD" V 10640 2640 50  0001 C CNN
 F 3 "~" H 10600 2650 50  0001 C CNN
 	1    10600 2650
@@
 Connection ~ 6800 2400
 Text GLabel 7850 2400 2    50   Input ~ 0
-12P
++12P
 $EndSCHEMATC
