File: power_alec/buck.kicad_pcb (KiCad board)
At the start: 4 copper layers, 35 parts, among them J8 Conn_01x01, J9 Conn_01x01, Q1 Q_PMOS_GDS

Commit message: updated library
Parts:
- moved BC1 415.4 mm to (115.0, 60.7)
- moved BC2 415.4 mm to (115.2, 102.8)
- moved BC3 415.4 mm to (187.8, 60.6)
- moved BC4 415.4 mm to (195.2, 129.6)
- moved C13 415.4 mm to (101.7, 101.2)
- moved C14 415.4 mm to (101.2, 117.2)
- moved C15 415.4 mm to (182.5, 96.2)
- moved C16 415.4 mm to (181.5, 78.2)
- moved C17 415.4 mm to (181.5, 87.2)
- moved C18 415.4 mm to (183.4, 115.2)
- moved C19 415.4 mm to (187.0, 115.2)
- moved D1 415.4 mm to (101.7, 95.2)
- moved D2 415.4 mm to (198.8, 55.6)
- moved D4 415.4 mm to (114.9, 53.1)
- moved D5 415.4 mm to (149.3, 55.3)
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Routing:
- net +5V: track 6.96 -> 18.5 mm
- net GNDS: track 10.4 -> 21.4 mm
