File: esc_breakout/esc_breakout.kicad_pcb (KiCad board)
At the start: 4 copper layers, 78 parts, among them J1 Conn_01x03_Female, J2 Conn_01x03_Female, J3 Conn_01x03_Female, J4 Conn_01x03_Female, J5 Conn_01x03_Female, J6 Conn_01x03_Female, U1 PIC16F15323, U10 TSC888, U11 TSC888, U12 TSC888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

Commit message: updated library
Parts:
- moved J4 33.6 mm to (238.8, 68.1)
- moved J5 33.6 mm to (238.9, 99.6)
- moved J6 33.5 mm to (238.8, 124.8)
- moved J1 32.9 mm to (56.0, 81.5)
- moved J3 32.4 mm to (56.5, 136.0)
- moved J2 32.2 mm to (56.1, 109.1)
- moved R3 21.3 mm to (109.0, 117.7)
- moved ESC3 21.3 mm to (91.8, 121.0)
- moved ESC5 18.7 mm to (207.3, 112.8)
- moved R5 18.7 mm to (190.8, 113.1)
- moved R6 18.7 mm to (190.4, 138.0)
- moved ESC4 18.7 mm to (207.2, 86.3)
- moved R4 18.7 mm to (189.1, 87.0)
- moved ESC6 18.7 mm to (207.4, 138.0)
- moved R2 18.6 mm to (108.2, 92.4)
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Routing:
- net +12P: track 168.2 -> 63.4 mm, vias 15 -> 30
- net +5VP: track 24.6 -> 106.7 mm, vias 16 -> 19
- net Net-(ESC2-Pad1): track 39.3 -> 15.4 mm
- net Net-(ESC3-Pad1): track 38.4 -> 16.3 mm
- net Net-(ESC6-Pad1): track 31.8 -> 15.0 mm
- net Net-(ESC5-Pad1): track 31.9 -> 15.2 mm
- net Net-(ESC4-Pad1): track 29.8 -> 13.4 mm
- net /PWM3: track 72.9 -> 59.1 mm, vias 1 -> 0
- net /PWM2: track 69.8 -> 61.9 mm, vias 1 -> 0
- net GNDPWR: track 229.9 -> 222.1 mm, vias 18 -> 33
- net /CS3: track 25.7 -> 18.4 mm
- net /PWM6: track 62.3 -> 55.1 mm, vias 1 -> 0
- net /PWM5: track 60.9 -> 55.2 mm, vias 1 -> 0
- net /CS2: track 23.2 -> 18.3 mm
- net /PWM1: track 67.1 -> 62.5 mm, vias 1 -> 0
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Other:
- net class Default: trace_width 0.5 -> 0.25
