File: pi/pi.kicad_pcb (KiCad board)
At the start: 2 copper layers, 10 parts, among them U5 ADuM1250, U6 PI_ZERO

Commit message: updated library
Connections:
- R13 pad 1: 5VPI -> +5VP
- R14 pad 1: 5VPI -> +5VP
- U5 pad 8: 5VPI -> +5VP
Changed lines of the file:
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@@
     )
     (pad 1 smd roundrect (at -1.025 0 270) (size 1.15 1.4) (layers F.Cu F.Paste F.Mask) (roundrect_rratio 0.217391)
-      (net 5 5VPI))
+      (net 1 +5VP))
     (pad 2 smd roundrect (at 1.025 0 270) (size 1.15 1.4) (layers F.Cu F.Paste F.Mask) (roundrect_rratio 0.217391)
       (net 7 "Net-(R13-Pad2)"))
@@
       (net 8 "Net-(R14-Pad2)"))
     (pad 1 smd roundrect (at -1.025 0 90) (size 1.15 1.4) (layers F.Cu F.Paste F.Mask) (roundrect_rratio 0.217391)
-      (net 5 5VPI))
+      (net 1 +5VP))
     (model ${KISYS3DMOD}/Resistor_SMD.3dshapes/R_0805_2012Metric.wrl
       (at (xyz 0 0 0))
@@
       (net 7 "Net-(R13-Pad2)"))
     (pad 8 smd rect (at 3.7 -1.905) (size 1.75 0.55) (layers F.Cu F.Paste F.Mask)
-      (net 5 5VPI))
+      (net 1 +5VP))
     (model ${KISYS3DMOD}/Package_SO.3dshapes/SO-8_5.3x6.2mm_P1.27mm.wrl
       (at (xyz 0 0 0))
