File: pi/pi.sch (KiCad schematic (older format))
At the start: 10 parts, among them U5 ADuM1250, U6 PI_ZERO

Commit message: PCA symbol moved to sensor board
Parts:
- U6: footprint Connector_PinSocket_2.54mm:PinSocket_2x20_P2.54mm_Vertical -> rov:PI_ZERO
Changed lines of the file:
@@
 F 0 "U6" H 5950 3625 50  0000 C CNN
 F 1 "PI_ZERO" H 5950 3534 50  0000 C CNN
-F 2 "Connector_PinSocket_2.54mm:PinSocket_2x20_P2.54mm_Vertical" H 5700 3200 50  0001 C CNN
+F 2 "rov:PI_ZERO" H 5700 3200 50  0001 C CNN
 F 3 "" H 5700 3200 50  0001 C CNN
 	1    5950 2550

Commit message: updated library
Changed lines of the file:
@@
 EESchema Schematic File Version 4
-LIBS:backplane-cache
+LIBS:pi-cache
 EELAYER 26 0
 EELAYER END
 $Descr A4 11693 8268
 encoding utf-8
-Sheet 1 5
+Sheet 1 1
 Title ""
 Date ""
@@
 	1    0    0    -1
 $EndComp
-Text GLabel 4000 1700 2    50   Input ~ 0
-5VPI
 $Comp
 L power:+5VP #PWR0144
@@
 	3850 1800 4400 1800
 Connection ~ 4400 1800
-Text GLabel 4750 1600 2    50   Input ~ 0
-5VPI
 Wire Wire Line
 	3850 1900 4400 1900
@@
 Wire Wire Line
 	4400 1600 4750 1600
-Text GLabel 4750 2100 2    50   Input ~ 0
-5VPI
 Wire Wire Line
 	4750 2100 4400 2100
@@
 NoConn ~ 6850 3500
 NoConn ~ 6850 3600
+$Comp
+L power:+5VP #PWR0105
+U 1 1 5C29B2D9
+P 4000 1700
+F 0 "#PWR0105" H 4000 1550 50  0001 C CNN
+F 1 "+5VP" H 4015 1873 50  0000 C CNN
+F 2 "" H 4000 1700 50  0001 C CNN
+F 3 "" H 4000 1700 50  0001 C CNN
+	1    4000 1700
+	1    0    0    -1
+$EndComp
+$Comp
+L power:+5VP #PWR?
+U 1 1 5C29B442
+P 4750 1600
+F 0 "#PWR?" H 4750 1450 50  0001 C CNN
+F 1 "+5VP" H 4765 1773 50  0000 C CNN
+F 2 "" H 4750 1600 50  0001 C CNN
+F 3 "" H 4750 1600 50  0001 C CNN
+	1    4750 1600
+	1    0    0    -1
+$EndComp
+$Comp
+L power:+5VP #PWR?
+U 1 1 5C29C44D
+P 4750 2100
+F 0 "#PWR?" H 4750 1950 50  0001 C CNN
+F 1 "+5VP" H 4765 2273 50  0000 C CNN
+F 2 "" H 4750 2100 50  0001 C CNN
+F 3 "" H 4750 2100 50  0001 C CNN
+	1    4750 2100
+	1    0    0    -1
+$EndComp
 $EndSCHEMATC
