File: sensor_suite/_saved_sensor_suite.sch (KiCad schematic (older format))
At the start: 11 parts, among them J1 Bar02, J2 Conn_01x02, J3 Conn_01x02, J4 LSM303, U1 MAX6581, U2 LM3480-3.3

Commit message: PCA symbol moved to sensor board
Parts:
- removed J1: Bar02, Connector_PinHeader_2.54mm:PinHeader_1x04_P2.54mm_Vertical, symbol Connector_Generic:Conn_01x04
- removed J2: Conn_01x02, Connector_JST:JST_EH_B02B-EH-A_1x02_P2.50mm_Vertical, symbol Connector_Generic:Conn_01x02
- removed J4: LSM303, Connector_PinHeader_2.54mm:PinHeader_1x08_P2.54mm_Vertical, symbol Connector_Generic:Conn_01x08
- added J?: Conn_01x02, Connector_JST:JST_EH_B02B-EH-A_1x02_P2.50mm_Vertical, symbol Connector_Generic:Conn_01x02
- added J?: LSM303, Connector_PinHeader_2.54mm:PinHeader_1x08_P2.54mm_Vertical, symbol Connector_Generic:Conn_01x08
- added J?: Bar02, Connector_PinHeader_2.54mm:PinHeader_1x04_P2.54mm_Vertical, symbol Connector_Generic:Conn_01x04
- added J?: Conn_02x15_Top_Bottom, symbol Connector_Generic:Conn_02x15_Top_Bottom
- added MH? (x4): MountingHole, Mounting_Holes:MountingHole_3.2mm_M3, symbol Mechanical:MountingHole
- renumbered C4 to C?, C5 to C?, C2 to C?, C1 to C?, C3 to C?, J3 to J?, U2 to U?, U1 to U?
Connections:
- net labels added: +5P, +5V, PWM0, PWM1, PWM2, PWM3, PWM4, PWM5
- wire segments 60 -> 98
- no-connect marks 3 -> 4

Commit message: updated library
Parts:
- J2: renamed from J?; footprint (none) -> rov:PCA9685
- J5: renamed from J?; footprint Connector_PinHeader_2.54mm:PinHeader_1x08_P2.54mm_Vertical -> rov:LSM303
- gave numbers to parts that had none: 14
Connections:
- net labels added: +5VP, GNDPWR
- net labels removed: +12P, +5P, +5V
- wire segments 98 -> 100

Commit message: Sensor Board
Parts:
- removed J2: Conn_02x15_Top_Bottom, rov:PCA9685, symbol Connector_Generic:Conn_02x15_Top_Bottom
- removed MH1, MH2, MH3, MH4: MountingHole, Mounting_Holes:MountingHole_3.2mm_M3, symbol Mechanical:MountingHole
- removed U1: MAX6581, Package_DFN_QFN:QFN-20-1EP_5x5mm_P0.65mm_EP3.35x3.35mm, symbol ROV:MAX6581
- added C10, C9: 100 pF, 100 pF, symbol Device:C_Small
- added C6, C7, C8: 100 pF, symbol Device:C_Small
- added CN1: 609-3634-ND, ROV:609-3634-ND, symbol rov:609-3634-ND
- added J2: Conn_02x10_Counter_Clockwise, ROV:PCA9685, symbol Connector_Generic:Conn_02x10_Counter_Clockwise
- added J6: Conn_02x20_Counter_Clockwise, Connector_PinHeader_2.54mm:PinHeader_2x20_P2.54mm_Vertical, symbol Connector_Generic:Conn_02x20_Counter_Clockwise
- added R1, R2: 10k, symbol Device:R_Small
- added U1: MAX6581, symbol rov:MAX6581
- J5: footprint rov:LSM303 -> Connector_PinHeader_2.54mm:PinHeader_1x08_P2.54mm_Vertical
Connections:
- net labels added: +12P, PWM_0, PWM_1, PWM_10, PWM_11, PWM_12, PWM_13, PWM_14, PWM_15, PWM_2, PWM_3, PWM_4, PWM_5, PWM_6, PWM_7, PWM_8, PWM_9
- net labels removed: GND, PWM0, PWM1, PWM2, PWM3, PWM4, PWM5
- wire segments 100 -> 131
- no-connect marks 4 -> 5
